File: board/eagle/tama.brd (EAGLE design)
At the start: 100 x 50 mm, 35 parts, among them J1 AVR_SPI_PRG_6NS

Commit message: Added an SMT crystal (not connected yet). Unsure if this is the right package...
Parts:
- added C4, C5: (no value), SparkFun:0805
- added Q1: (no value), crystal:CTS406
Connections:
- new net N$25: C4.2, Q1.3
- new net N$26: C5.1, U$4.16
- new net N$27: C5.2, Q1.1
- new net N$28: C4.1, U$4.17
Routing:
- net D-: track 58.0 -> 61.2 mm
Changed lines of the file:
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@@
 <?xml version="1.0" encoding="utf-8"?>
 <!DOCTYPE eagle SYSTEM "eagle.dtd">
-<eagle version="6.5.0">
+<eagle version="6.4">
 <drawing>
 <settings>
@@
 <grid distance="10" unitdist="mil" unit="mil" style="lines" multiple="1" display="yes" altdistance="0.025" altunitdist="inch" altunit="inch"/>
 <layers>
-<layer number="1" name="Top" color="4" fill="1" visible="no" active="yes"/>
-<layer number="16" name="Bottom" color="1" fill="1" visible="no" active="yes"/>
-<layer number="17" name="Pads" color="2" fill="1" visible="no" active="yes"/>
-<layer number="18" name="Vias" color="2" fill="1" visible="no" active="yes"/>
-<layer number="19" name="Unrouted" color="6" fill="1" visible="no" active="yes"/>
-<layer number="20" name="Dimension" color="15" fill="1" visible="no" active="yes"/>
+<layer number="1" name="Top" color="4" fill="1" visible="yes" active="yes"/>
+<layer number="16" name="Bottom" color="1" fill="1" visible="yes" active="yes"/>
+<layer number="17" name="Pads" color="2" fill="1" visible="yes" active="yes"/>
+<layer number="18" name="Vias" color="2" fill="1" visible="yes" active="yes"/>
+<layer number="19" name="Unrouted" color="6" fill="1" visible="yes" active="yes"/>
+<layer number="20" name="Dimension" color="15" fill="1" visible="yes" active="yes"/>
 <layer number="21" name="tPlace" color="5" fill="1" visible="no" active="yes"/>
-<layer number="22" name="bPlace" color="7" fill="1" visible="yes" active="yes"/>
-<layer number="23" name="tOrigins" color="15" fill="1" visible="no" active="yes"/>
+<layer number="22" name="bPlace" color="7" fill="1" visible="no" active="yes"/>
+<layer number="23" name="tOrigins" color="15" fill="1" visible="yes" active="yes"/>
 <layer number="24" name="bOrigins" color="15" fill="1" visible="no" active="yes"/>
 <layer number="25" name="tNames" color="7" fill="1" visible="no" active="yes"/>
@@
 <layer number="28" name="bValues" color="7" fill="1" visible="no" active="yes"/>
 <layer number="29" name="tStop" color="7" fill="3" visible="no" active="yes"/>
-<layer number="30" name="bStop" color="7" fill="6" visible="yes" active="yes"/>
+<layer number="30" name="bStop" color="7" fill="6" visible="no" active="yes"/>
 <layer number="31" name="tCream" color="7" fill="4" visible="no" active="yes"/>
 <layer number="32" name="bCream" color="7" fill="5" visible="no" active="yes"/>
@@
 <layer number="49" name="Reference" color="7" fill="1" visible="no" active="yes"/>
 <layer number="50" name="dxf" color="12" fill="1" visible="no" active="no"/>
-<layer number="51" name="tDocu" color="7" fill="1" visible="no" active="yes"/>
-<layer number="52" name="bDocu" color="7" fill="1" visible="no" active="yes"/>
+<layer number="51" name="tDocu" color="7" fill="1" visible="yes" active="yes"/>
+<layer number="52" name="bDocu" color="7" fill="1" visible="yes" active="yes"/>
 <layer number="53" name="tGND_GNDA" color="7" fill="1" visible="no" active="no"/>
 <layer number="54" name="bGND_GNDA" color="7" fill="1" visible="no" active="no"/>
@@
 <element name="C2" library="rcl" package="C1206" value="100n" x="56.0556" y="30.9152" smashed="yes"/>
 <element name="J1" library="SparkFun-Connectors" package="2X3-NS" value="AVR_SPI_PRG_6NS" x="82" y="4" smashed="yes"/>
+<element name="Q1" library="crystal" package="CTS406" value="" x="43.434" y="30.48">
+<attribute name="OC_NEWARK" value="unknown" x="43.434" y="30.48" size="1.778" layer="27" display="off"/>
+<attribute name="MPN" value="" x="43.434" y="30.48" size="1.778" layer="27" display="off"/>
+<attribute name="MF" value="" x="43.434" y="30.48" size="1.778" layer="27" display="off"/>
+<attribute name="OC_FARNELL" value="unknown" x="43.434" y="30.48" size="1.778" layer="27" display="off"/>
+</element>
+<element name="C4" library="SparkFun" package="0805" value="" x="50.292" y="30.48"/>
+<element name="C5" library="SparkFun" package="0805" value="" x="33.782" y="32.004"/>
 </elements>
 <signals>
@@
 <wire x1="56.900003125" y1="13.800003125" x2="63.400003125" y2="13.800003125" width="0.4064" layer="16"/>
 <wire x1="54.300003125" y1="13.800003125" x2="56.900003125" y2="13.800003125" width="0.4064" layer="1"/>
-<wire x1="40.600003125" y1="27.500003125" x2="54.300003125" y2="13.800003125" width="0.4064" layer="16"/>
-<wire x1="40.600003125" y1="35.600003125" x2="40.600003125" y2="27.500003125" width="0.4064" layer="1"/>
+<wire x1="52.538003125" y1="31.818003125" x2="54.300003125" y2="13.800003125" width="0.4064" layer="16"/>
+<wire x1="40.600003125" y1="35.600003125" x2="52.538003125" y2="31.818003125" width="0.4064" layer="1"/>
 <wire x1="40.600003125" y1="38.900003125" x2="40.600003125" y2="35.600003125" width="0.4064" layer="16"/>
 <wire x1="40.400003125" y1="38.900003125" x2="40.600003125" y2="38.900003125" width="0.4064" layer="16"/>
@@
 <via x="56.900003125" y="13.800003125" extent="1-16" drill="0.6096"/>
 <via x="54.300003125" y="13.800003125" extent="1-16" drill="0.6096"/>
-<via x="40.600003125" y="27.500003125" extent="1-16" drill="0.6096"/>
+<via x="52.538003125" y="31.818003125" extent="1-16" drill="0.6096"/>
 <via x="40.600003125" y="35.600003125" extent="1-16" drill="0.6096"/>
 <via x="40.400003125" y="38.900003125" extent="1-16" drill="0.6096"/>
@@
 <wire x1="7.200003125" y1="17.300003125" x2="7.1326" y2="17.3252" width="0.4064" layer="1"/>
 </signal>
+<signal name="N$25">
+<contactref element="Q1" pad="3"/>
+<contactref element="C4" pad="2"/>
+<wire x1="45.634" y1="31.68" x2="51.192" y2="30.48" width="0" layer="19" extent="1-1"/>
+</signal>
+<signal name="N$26">
+<contactref element="U$4" pad="16"/>
+<contactref element="C5" pad="1"/>
+<wire x1="32.882" y1="32.004" x2="43.6926" y2="22.9942" width="0" layer="19" extent="1-1"/>
+</signal>
+<signal name="N$27">
+<contactref element="Q1" pad="1"/>
+<contactref element="C5" pad="2"/>
+<wire x1="41.234" y1="29.28" x2="34.682" y2="32.004" width="0" layer="19" extent="1-1"/>
+</signal>
+<signal name="N$28">
+<contactref element="U$4" pad="17"/>
+<contactref element="C4" pad="1"/>
+<wire x1="49.392" y1="30.48" x2="42.8926" y2="22.9942" width="0" layer="19" extent="1-1"/>
+</signal>
 </signals>

Commit message: Redid the crystal based on the datasheet. (See pg 30 of the preliminary ATmega32U4 datasheet, doc7766.pdf)
Parts:
- C4, C5: value (none) -> 22pF
- Q1: value (none) -> 16Mhz
- moved C5 14.1 mm to (47.5, 28.7), turned to 270 degrees
- moved C4 12.1 mm to (38.4, 28.7), turned to 90 degrees
- moved Q1 1.37 mm to (42.9, 29.2), turned to 180 degrees
- turned R16 to 180 degrees
Connections:
- removed net N$27: C5.2, Q1.1
- removed net N$28: C4.1, U$4.17
- net GND: now also C4.2, C5.2
- net N$25: now also C4.1, U$4.17; no longer C4.2
- net N$26: now also Q1.1
Routing:
- net D-: track 61.2 -> 41.0 mm, vias 6 -> 2
- net N$26: track 0.00 -> 12.0 mm
- net IO11*: track 47.0 -> 59.0 mm
- net GND: track 88.2 -> 99.3 mm
- net N$25: track 0.00 -> 9.76 mm
- net RD-: track 28.0 -> 20.6 mm
- net V33: track 201.3 -> 207.2 mm
- net N$6: track 36.5 -> 41.9 mm, vias 2 -> 1
- net N$13: track 42.8 -> 44.8 mm
